File: power.kicad_sch (KiCad schematic)
At the start: 24 parts, among them J4 USB_C_Receptacle_USB2.0, J5 Conn_01x05, U2 Protection_SRV05-4A, U3 LMR33630BDDA, U6 XC6206P332MR

Commit message: connect spi and uart to pi interface
we'll even have jumpers for being the hat or the baseboard for uart...

need to re-open modus to find new pins for i2c...
Other:
- note added: "Classic JBT Marel CAN connector"
Changed lines of the file:
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@@
 	(generator_version "10.0")
 	(paper "A4")
+	(text "Classic JBT Marel CAN connector"
+		(exclude_from_sim no)
+		(at 40.132 144.78 0)
+		(effects
+			(font
+				(size 1.27 1.27)
+			)
+		)
+	)
 	(text "mixed size here is to get a perfect\n4:1 ratio for 5V in JLC basic resistors"
 		(exclude_from_sim no)
